File: ESP Updater/ESP Updater.brd (EAGLE design)
At the start: 38 x 24 mm, 24 parts, among them J1 DX07S016JA1R1500, J2 52852-0670, Q1 MMBT2222, Q2 MMBT2222, U1 CP2104, U2 AMS1117-3.3

Commit message: Update
Parts:
- added C7: 0.1uF, rcl:C0603
- C1: value 10uF -> 1uF
- moved C1 7.38 mm to (14.7, 9.60), turned to 90 degrees
- moved C5 2.62 mm to (20.0, 5.70)
Connections:
- net 3.3: now also C7.1
- net GND: now also C7.2
Routing:
- net 3.3: track 123.3 -> 135.4 mm, vias 3 -> 4
- net GND: track 40.9 -> 51.5 mm, vias 5 -> 6
- net N$8: track 5.48 -> 2.95 mm
- net VCC: track 26.9 -> 27.7 mm
- net D-: track 21.2 -> 21.8 mm
