File: ESP Updater/ESP Updater.sch (EAGLE design)
At the start: 24 parts, among them J1 DX07S016JA1R1500, J2 52852-0670, Q1 MMBT2222, Q2 MMBT2222, U1 CP2104, U2 AMS1117-3.3

Commit message: Update
Parts:
- added C7: 0.1uF, rcl:C-EUC0603
- C1: value 10uF -> 1uF
Connections:
- net 3.3: now also C7.1
- net GND: now also C7.2
Changed lines of the file:
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@@
 <part name="P+1" library="supply1" library_urn="urn:adsk.eagle:library:371" deviceset="VCC" device=""/>
 <part name="GND3" library="supply1" library_urn="urn:adsk.eagle:library:371" deviceset="GND" device=""/>
-<part name="C1" library="0805YC103J4T2A" library_urn="urn:adsk.eagle:library:37164964" deviceset="0805YC103J4T2A" device="" package3d_urn="urn:adsk.eagle:package:37164967/2" value="10uF"/>
+<part name="C1" library="0805YC103J4T2A" library_urn="urn:adsk.eagle:library:37164964" deviceset="0805YC103J4T2A" device="" package3d_urn="urn:adsk.eagle:package:37164967/2" value="1uF"/>
 <part name="GND4" library="supply1" library_urn="urn:adsk.eagle:library:371" deviceset="GND" device=""/>
 <part name="P+2" library="supply1" library_urn="urn:adsk.eagle:library:371" deviceset="VCC" device=""/>
@@
 <part name="C5" library="0805YC103J4T2A" library_urn="urn:adsk.eagle:library:37164964" deviceset="0805YC103J4T2A" device="" package3d_urn="urn:adsk.eagle:package:37164967/2" value="4.7uF"/>
 <part name="GND13" library="supply1" library_urn="urn:adsk.eagle:library:371" deviceset="GND" device=""/>
+<part name="C7" library="rcl" library_urn="urn:adsk.eagle:library:334" deviceset="C-EU" device="C0603" package3d_urn="urn:adsk.eagle:package:23616/2" value="0.1uF"/>
 </parts>
 <sheets>
@@
 <attribute name="VALUE" x="187.96" y="177.8" size="1.778" layer="96"/>
 </instance>
+<instance part="C7" gate="G$1" x="193.04" y="220.98" smashed="yes">
+<attribute name="NAME" x="194.564" y="221.361" size="1.778" layer="95"/>
+<attribute name="VALUE" x="194.564" y="216.281" size="1.778" layer="96"/>
+</instance>
 </instances>
 <busses>
@@
 <pinref part="GND4" gate="1" pin="GND"/>
 <junction x="182.88" y="215.9"/>
+<pinref part="C7" gate="G$1" pin="2"/>
+<wire x1="182.88" y1="215.9" x2="193.04" y2="215.9" width="0.1524" layer="91"/>
 </segment>
 <segment>
@@
 <pinref part="U1" gate="G$1" pin="VDD"/>
 <wire x1="241.3" y1="243.84" x2="243.84" y2="243.84" width="0.1524" layer="91"/>
-<wire x1="243.84" y1="243.84" x2="243.84" y2="251.46" width="0.1524" layer="91"/>
-<label x="243.84" y="251.46" size="1.778" layer="95"/>
+<wire x1="243.84" y1="243.84" x2="243.84" y2="256.54" width="0.1524" layer="91"/>
+<label x="243.84" y="256.54" size="1.778" layer="95"/>
 <pinref part="U1" gate="G$1" pin="VIO"/>
 <wire x1="241.3" y1="241.3" x2="243.84" y2="241.3" width="0.1524" layer="91"/>
@@
 <segment>
 <pinref part="U1" gate="G$1" pin="REGIN"/>
-<wire x1="200.66" y1="226.06" x2="182.88" y2="226.06" width="0.1524" layer="91"/>
+<wire x1="200.66" y1="226.06" x2="193.04" y2="226.06" width="0.1524" layer="91"/>
 <pinref part="C1" gate="G$1" pin="2"/>
+<wire x1="193.04" y1="226.06" x2="182.88" y2="226.06" width="0.1524" layer="91"/>
 <wire x1="182.88" y1="226.06" x2="182.88" y2="223.52" width="0.1524" layer="91"/>
 <wire x1="182.88" y1="226.06" x2="172.72" y2="226.06" width="0.1524" layer="91"/>
@@
 <junction x="182.88" y="223.52"/>
 <junction x="200.66" y="226.06"/>
+<pinref part="C7" gate="G$1" pin="1"/>
+<wire x1="193.04" y1="223.52" x2="193.04" y2="226.06" width="0.1524" layer="91"/>
+<junction x="193.04" y="226.06"/>
 </segment>
 <segment>
@@
 packages will not be understood (or retained) with this version.
 </note>
+<note version="8.4" severity="warning">
+Since Version 8.4, EAGLE supports properties for SPICE simulation.
+Probes in schematics and SPICE mapping objects found in parts and library devices
+will not be understood with this version. Update EAGLE to the latest version
+for full support of SPICE simulation.
+</note>
 </compatibility>
