File: Encoder/ESP8266 Encoder.brd (EAGLE design)
At the start: 44.5 x 38 mm, 15 parts, among them J2 52745-0697, J3 TB004-508-02BE, U1 ENCODER90

Commit message: Update
Parts:
- removed J2: 52745-0697, 52745-0697:0527450697
- removed JP1: (no value), pinhead:1X06
- added J1: 52852-0670, 52852-0670:528520670
- moved R7 4.12 mm to (34.6, 5.30)
- moved R2 3.16 mm to (34.6, 8.63)
Connections:
- net GND: now also J1.6; no longer J2.6, JP1.6
- net GPIO0: now also J1.3; no longer J2.3, JP1.3
- net RESET: now also J1.2; no longer J2.2, JP1.2
- net RX: now also J1.5; no longer J2.5, JP1.5
- net TX: now also J1.4; no longer J2.4, JP1.4
- net VCC: now also J1.1; no longer J2.1, JP1.1
Routing:
- net RX: track 64.9 -> 24.7 mm
- net TX: track 56.3 -> 24.7 mm, vias 2 -> 1
- net GPIO0: track 43.8 -> 26.8 mm, vias 2 -> 1
- net RESET: track 58.1 -> 41.4 mm, vias 4 -> 2
- net VCC: track 88.1 -> 76.4 mm, vias 4 -> 2
- net GPIO2: track 11.1 -> 13.3 mm
Other:
- board size 44.5 x 38 mm -> 44.5 x 40.5 mm
- board text removed: "1"
- board text removed: "6"
