File: Encoder/ESP8266 Encoder.sch (EAGLE design)
At the start: 15 parts, among them J2 52745-0697, J3 TB004-508-02BE, U1 ENCODER90

Commit message: Update
Parts:
- removed J2: 52745-0697, 52745-0697:52745-0697
- removed JP1: (no value), pinhead:PINHD-1X6
- added J1: 52852-0670, 52852-0670:52852-0670
Connections:
- net GND: now also J1.6; no longer J2.6, JP1.6
- net GPIO0: now also J1.3; no longer J2.3, JP1.3
- net RESET: now also J1.2; no longer J2.2, JP1.2
- net RX: now also J1.5; no longer J2.5, JP1.5
- net TX: now also J1.4; no longer J2.4, JP1.4
- net VCC: now also J1.1; no longer J2.1, JP1.1
Other:
- moved on the sheet: J3
Changed lines of the file:
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@@
 <part name="P+3" library="supply1" library_urn="urn:adsk.eagle:library:371" deviceset="VCC" device=""/>
 <part name="P+4" library="supply1" library_urn="urn:adsk.eagle:library:371" deviceset="VCC" device=""/>
-<part name="JP1" library="pinhead" library_urn="urn:adsk.eagle:library:325" deviceset="PINHD-1X6" device="" package3d_urn="urn:adsk.eagle:package:22472/2"/>
-<part name="P+5" library="supply1" library_urn="urn:adsk.eagle:library:371" deviceset="VCC" device=""/>
-<part name="GND4" library="supply1" library_urn="urn:adsk.eagle:library:371" deviceset="GND" device=""/>
 <part name="GND5" library="supply1" library_urn="urn:adsk.eagle:library:371" deviceset="GND" device=""/>
 <part name="GND6" library="supply1" library_urn="urn:adsk.eagle:library:371" deviceset="GND" device=""/>
@@
 <part name="P+8" library="supply1" library_urn="urn:adsk.eagle:library:371" deviceset="VCC" device=""/>
 <part name="FRAME2" library="frames" library_urn="urn:adsk.eagle:library:229" deviceset="FRAME_A_L" device=""/>
-<part name="J2" library="52745-0697" library_urn="urn:adsk.eagle:library:39835023" deviceset="52745-0697" device="" package3d_urn="urn:adsk.eagle:package:39835026/2"/>
 <part name="J3" library="TB004-508-02BE" library_urn="urn:adsk.eagle:library:39835436" deviceset="TB004-508-02BE" device="" package3d_urn="urn:adsk.eagle:package:39835439/2"/>
 <part name="GND9" library="supply1" library_urn="urn:adsk.eagle:library:371" deviceset="GND" device=""/>
@@
 <part name="R7" library="RC0805FR-07330RL" library_urn="urn:adsk.eagle:library:37164869" deviceset="RC0805FR-07330RL" device="" package3d_urn="urn:adsk.eagle:package:37164874/2" value="10K"/>
 <part name="P+10" library="supply1" library_urn="urn:adsk.eagle:library:371" deviceset="VCC" device=""/>
+<part name="J1" library="52852-0670" library_urn="urn:adsk.eagle:library:39834973" deviceset="52852-0670" device="" package3d_urn="urn:adsk.eagle:package:39834977/2"/>
 </parts>
 <sheets>
@@
 <attribute name="VALUE" x="-76.2" y="-20.32" size="1.778" layer="96" rot="R90"/>
 </instance>
-<instance part="JP1" gate="A" x="-78.74" y="35.56" smashed="yes">
-<attribute name="NAME" x="-85.09" y="46.355" size="1.778" layer="95"/>
-<attribute name="VALUE" x="-85.09" y="25.4" size="1.778" layer="96"/>
-</instance>
-<instance part="P+5" gate="VCC" x="-91.44" y="50.8" smashed="yes">
-<attribute name="VALUE" x="-86.36" y="53.34" size="1.778" layer="96" rot="R180"/>
-</instance>
-<instance part="GND4" gate="1" x="-91.44" y="25.4" smashed="yes">
-<attribute name="VALUE" x="-93.98" y="22.86" size="1.778" layer="96"/>
-</instance>
 <instance part="GND5" gate="1" x="35.56" y="10.16" smashed="yes">
 <attribute name="VALUE" x="33.02" y="7.62" size="1.778" layer="96"/>
@@
 <attribute name="DRAWING_NAME" x="38.1" y="-57.15" size="2.54" layer="94"/>
 </instance>
-<instance part="J2" gate="G$1" x="-76.2" y="43.18" smashed="yes"/>
-<instance part="J3" gate="G$1" x="-111.76" y="96.52" smashed="yes" rot="R180">
-<attribute name="NAME" x="-113.03" y="93.98" size="1.778" layer="95" rot="R180" align="center-left"/>
+<instance part="J3" gate="G$1" x="-109.22" y="96.52" smashed="yes" rot="R180">
+<attribute name="NAME" x="-110.49" y="93.98" size="1.778" layer="95" rot="R180" align="center-left"/>
 </instance>
 <instance part="GND9" gate="1" x="-55.88" y="27.94" smashed="yes">
@@
 <attribute name="VALUE" x="-43.18" y="-20.32" size="1.778" layer="96" rot="R90"/>
 </instance>
+<instance part="J1" gate="G$1" x="-88.9" y="43.18" smashed="yes"/>
 </instances>
 <busses>
@@
 <segment>
 <pinref part="PS2" gate="G$1" pin="VAC_IN(L)"/>
-<wire x1="-111.76" y1="99.06" x2="-96.52" y2="99.06" width="0.1524" layer="91"/>
+<wire x1="-109.22" y1="99.06" x2="-96.52" y2="99.06" width="0.1524" layer="91"/>
 <wire x1="-96.52" y1="99.06" x2="-96.52" y2="106.68" width="0.1524" layer="91"/>
 <wire x1="-96.52" y1="106.68" x2="-86.36" y2="106.68" width="0.1524" layer="91"/>
@@
 <segment>
 <pinref part="PS2" gate="G$1" pin="VAC_IN(N)"/>
-<wire x1="-111.76" y1="96.52" x2="-86.36" y2="96.52" width="0.1524" layer="91"/>
+<wire x1="-109.22" y1="96.52" x2="-86.36" y2="96.52" width="0.1524" layer="91"/>
 <pinref part="J3" gate="G$1" pin="1"/>
 </segment>
@@
 </segment>
 <segment>
-<pinref part="JP1" gate="A" pin="1"/>
-<pinref part="P+5" gate="VCC" pin="VCC"/>
-<wire x1="-81.28" y1="43.18" x2="-91.44" y2="43.18" width="0.1524" layer="91"/>
-<wire x1="-91.44" y1="43.18" x2="-91.44" y2="48.26" width="0.1524" layer="91"/>
-</segment>
-<segment>
 <pinref part="R4" gate="G$1" pin="2"/>
 <pinref part="P+6" gate="VCC" pin="VCC"/>
@@
 </segment>
 <segment>
-<pinref part="J2" gate="G$1" pin="1"/>
-<pinref part="P+9" gate="VCC" pin="VCC"/>
-</segment>
-<segment>
 <pinref part="R7" gate="G$1" pin="2"/>
 <wire x1="-40.64" y1="-25.4" x2="-40.64" y2="-20.32" width="0.1524" layer="91"/>
 <pinref part="P+10" gate="VCC" pin="VCC"/>
 </segment>
+<segment>
+<pinref part="P+9" gate="VCC" pin="VCC"/>
+<pinref part="J1" gate="G$1" pin="1"/>
+<wire x1="-68.58" y1="43.18" x2="-55.88" y2="43.18" width="0.1524" layer="91"/>
+</segment>
 </net>
 <net name="GND" class="0">
@@
 <pinref part="R3" gate="G$1" pin="1"/>
 <pinref part="GND3" gate="1" pin="GND"/>
-</segment>
-<segment>
-<pinref part="JP1" gate="A" pin="6"/>
-<pinref part="GND4" gate="1" pin="GND"/>
-<wire x1="-81.28" y1="30.48" x2="-91.44" y2="30.48" width="0.1524" layer="91"/>
-<wire x1="-91.44" y1="30.48" x2="-91.44" y2="27.94" width="0.1524" layer="91"/>
 </segment>
 <segment>
@@
 </segment>
 <segment>
-<pinref part="J2" gate="G$1" pin="6"/>
 <pinref part="GND9" gate="1" pin="GND"/>
+<pinref part="J1" gate="G$1" pin="6"/>
+<wire x1="-68.58" y1="30.48" x2="-55.88" y2="30.48" width="0.1524" layer="91"/>
 </segment>
 </net>
@@
 </segment>
 <segment>
-<pinref part="JP1" gate="A" pin="2"/>
-<wire x1="-81.28" y1="40.64" x2="-101.6" y2="40.64" width="0.1524" layer="91"/>
-<label x="-101.6" y="40.64" size="1.778" layer="95"/>
-</segment>
-<segment>
-<pinref part="J2" gate="G$1" pin="2"/>
-<wire x1="-55.88" y1="40.64" x2="-38.1" y2="40.64" width="0.1524" layer="91"/>
+<wire x1="-68.58" y1="40.64" x2="-38.1" y2="40.64" width="0.1524" layer="91"/>
 <label x="-45.72" y="40.64" size="1.778" layer="95"/>
+<pinref part="J1" gate="G$1" pin="2"/>
 </segment>
 <segment>
@@
 </segment>
 <segment>
-<pinref part="JP1" gate="A" pin="3"/>
-<wire x1="-81.28" y1="38.1" x2="-101.6" y2="38.1" width="0.1524" layer="91"/>
-<label x="-101.6" y="38.1" size="1.778" layer="95"/>
-</segment>
-<segment>
-<pinref part="J2" gate="G$1" pin="3"/>
-<wire x1="-55.88" y1="38.1" x2="-38.1" y2="38.1" width="0.1524" layer="91"/>
+<wire x1="-68.58" y1="38.1" x2="-38.1" y2="38.1" width="0.1524" layer="91"/>
 <label x="-45.72" y="38.1" size="1.778" layer="95"/>
+<pinref part="J1" gate="G$1" pin="3"/>
 </segment>
 </net>
@@
 </segment>
 <segment>
-<pinref part="JP1" gate="A" pin="4"/>
-<wire x1="-81.28" y1="35.56" x2="-101.6" y2="35.56" width="0.1524" layer="91"/>
-<label x="-101.6" y="35.56" size="1.778" layer="95"/>
-</segment>
-<segment>
-<pinref part="J2" gate="G$1" pin="4"/>
-<wire x1="-55.88" y1="35.56" x2="-38.1" y2="35.56" width="0.1524" layer="91"/>
+<wire x1="-68.58" y1="35.56" x2="-38.1" y2="35.56" width="0.1524" layer="91"/>
 <label x="-45.72" y="35.56" size="1.778" layer="95"/>
+<pinref part="J1" gate="G$1" pin="4"/>
 </segment>
 </net>
@@
 </segment>
 <segment>
-<pinref part="JP1" gate="A" pin="5"/>
-<wire x1="-81.28" y1="33.02" x2="-101.6" y2="33.02" width="0.1524" layer="91"/>
-<label x="-101.6" y="33.02" size="1.778" layer="95"/>
-</segment>
-<segment>
-<pinref part="J2" gate="G$1" pin="5"/>
-<wire x1="-55.88" y1="33.02" x2="-38.1" y2="33.02" width="0.1524" layer="91"/>
+<wire x1="-68.58" y1="33.02" x2="-38.1" y2="33.02" width="0.1524" layer="91"/>
 <label x="-45.72" y="33.02" size="1.778" layer="95"/>
-</segment>
-</net>
+<pinref part="J1" gate="G$1" pin="5"/>
+</segment>
+</net>
