File: Thermometer/ESP Thermometer.brd (EAGLE design)
At the start: 39.5 x 34 mm, 13 parts, among them J1 TB006-508-02BE, J2 52852-0670

Commit message: Update
Parts:
- removed HM1: HTU21D, HTU21D:SON100P300X300X100-7N
- added C2: 0.1uF, 0805YC103J4T2A:CAPC2012X94N
- added IC1: HS3003, HS3003:HS3004
- R5, R6: value 4.7K -> 2.2K
- moved C1 1.75 mm to (32.5, 30.0)
- moved R3 1.00 mm to (26.5, 22.0)
- moved R5 1.00 mm to (25.4, 28.2)
- moved R6 1.00 mm to (25.4, 31.4)
Connections:
- new net N$3: C1.1, IC1.3
- net GND: now also C1.2, C2.1, IC1.6; no longer C1.1, HM1.2, HM1.7
- net SCK: now also IC1.1; no longer HM1.6
- net SDA: now also IC1.2; no longer HM1.1
- net VCC: now also C2.2, IC1.4; no longer C1.2, HM1.5
Routing:
- net N$3: track 0.00 -> 5.48 mm
- net SCK: track 39.5 -> 43.0 mm
- net GND: track 53.3 -> 50.2 mm, vias 3 -> 4
- net VCC: track 79.0 -> 76.2 mm
- net GPIO0: track 27.1 -> 25.7 mm
- net SDA: track 46.4 -> 45.2 mm
Other:
- outline, holes or cut-outs redrawn
