File: Thermometer/ESP Thermometer.sch (EAGLE design)
At the start: 13 parts, among them J1 TB006-508-02BE, J2 52852-0670

Commit message: Update
Parts:
- removed HM1: HTU21D, HTU21D:HTU21D
- added C2: 0.1uF, 0805YC103J4T2A:0805YC103J4T2A
- added IC1: HS3003, HS3003:HS3003
- R5, R6: value 4.7K -> 2.2K
Connections:
- new net N$3: C1.1, IC1.VC
- net GND: now also C1.2, C2.1, IC1.VSS; no longer C1.1, HM1.EP, HM1.GND
- net SCK: now also IC1.SCL; no longer HM1.SCK
- net SDA: now also IC1.SDA; no longer HM1.DATA
- net VCC: now also C2.2, IC1.VDD; no longer C1.2, HM1.VDD
Other:
- moved on the sheet: C1, R5
